File: tps54338-buck.kicad_sch (KiCad schematic)
At the start: 17 parts, among them J1 VIN, J2 VOUT, U1 TPS54338

Commit message: Add PCB layout, BOM, and assembly files for Seeed Fusion
- PCB layout with 2-layer board, GND pour on B.Cu, copper pours for
  VIN/SW/VOUT on F.Cu, in-pad GND vias
- Selectable output voltage via solder jumper resistor network
  (3.3V/5.1V/12.6V)
- BOM with sourced LCSC parts: TDK VLS6045AF-6R8M inductor,
  Yageo 75k/200k resistors, Murata caps
- Clean ERC (0 errors) and DRC (0 unconnected, excluded footprint
  clearance violations within U1)
- Mounting hole M2.5
- Custom board artwork

Co-Authored-By: Claude Opus 4.6 (1M context) <noreply@anthropic.com>
Parts:
- JP1, JP2, JP3: footprint (none) -> Jumper:SolderJumper-2_P1.3mm_Open_Pad1.0x1.5mm
- L1: value 5.6uH -> 6.8uH
- R3: value 190k -> 200k
Changed lines of the file:
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@@
 			)
 		)
-		(property "Footprint" ""
+		(property "Footprint" "Jumper:SolderJumper-2_P1.3mm_Open_Pad1.0x1.5mm"
 			(at 179.07 104.14 0)
 			(effects
@@
 			)
 		)
-		(property "Footprint" ""
+		(property "Footprint" "Jumper:SolderJumper-2_P1.3mm_Open_Pad1.0x1.5mm"
 			(at 179.07 95.25 0)
 			(effects
@@
 			)
 		)
-		(property "Value" "190k"
+		(property "Value" "200k"
 			(at 168.91 104.14 90)
 			(effects
@@
 			)
 		)
-		(property "Value" "5.6uH"
+		(property "Value" "6.8uH"
 			(at 216.154 66.548 90)
 			(effects
@@
 			)
 		)
-		(property "Footprint" ""
+		(property "Footprint" "Jumper:SolderJumper-2_P1.3mm_Open_Pad1.0x1.5mm"
 			(at 179.07 86.36 0)
 			(effects
